File: kicad/4017-leds.kicad_sch (KiCad schematic)
At the start: 8 parts, among them U4 4017

Commit message: Note BOM effects in different implementations
Other:
- note added: "KNOWN ISSUES: * non-digit output BOM ADDITION: 7"
Changed lines of the file:
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@@
     (stroke (width 0) (type default) (color 0 0 0 0))
+  )
+  (text "KNOWN ISSUES:\n* non-digit output\n\nBOM ADDITION: 7" (at 151.13 107.95 0)
+    (effects (font (size 1.27 1.27)) (justify left bottom))
   )
   (hierarchical_label "OSC" (shape input) (at 113.03 80.645 180)
